File: boards/eos/eos-atmega328p-board/hardware/eos-atmega328p-board.kicad_pcb (KiCad board)
At the start: 2 copper layers, 68.6 x 53.3 mm, 71 parts, among them J1 USB-C, J2 7-12V, J3 D0-D7, J4 D8-SCL, J5 POWER, J6 A0-A5, J7 ICSP, SW1 RESET, U1 USBLC6-2SC6, U10 SN74LVC1G07, U2 AP63205, U3 TPS2116, U4 AP2112K-3.3, U5 CH340C, U6 ATmega328P-AU, U7 SN74LVC1G17, U8 SN74LVC1G17, U9 SN74LVC1G17, Y1 16MHz

Commit message: fix(boards): rebuild EoS boards without vias in pads
Co-authored-by: Cursor <cursoragent@cursor.com>
Routing:
- net /A4_SDA: track 85.1 -> 66.2 mm, vias 1 -> 2
- net +5V: track 178.1 -> 162.1 mm, vias 6 -> 7
- net GND: track 348.7 -> 359.5 mm, vias 128 -> 125
- net /RESET: track 77.8 -> 87.1 mm
- net /A3: track 47.3 -> 38.0 mm
- net /A5_SCL: track 78.1 -> 69.1 mm
- net /D0: track 56.7 -> 52.4 mm
- net /VUSB: track 76.8 -> 72.9 mm
- net /D1: track 107.8 -> 103.9 mm
- net /D6: track 15.8 -> 12.5 mm
- net /D4: track 24.3 -> 25.9 mm
- net /D13: track 62.3 -> 63.1 mm
- net /A2: track 38.0 -> 37.4 mm
- net /D3: track 26.4 -> 27.0 mm
