File: boards/eos/eos-cm4-base/hardware/eos-cm4-base.kicad_pcb (KiCad board)
At the start: 4 copper layers, 90 x 80 mm, 46 parts, among them J1 CM4 1-100, J2 CM4 101-200, J3 USB-C, J4 USB-A, J5 TRJG0926HENL, J6 microSD, J7 GPIO, J8 FAN, J9 BOOT, Q1 BSS84, Q2 2N7002, SW1 RESET, U1 USBLC6-2SC6, U2 TPS2051C, U3 USBLC6-2SC6, U4 TPD4EUSB30, U5 TPD4EUSB30, U6 RT9742GGJ5, U7 TS3USB30E

Commit message: fix(boards): rebuild EoS boards without vias in pads
Co-authored-by: Cursor <cursoragent@cursor.com>
Routing:
- net /GPIO3: track 40.4 -> 55.6 mm
- net /GPIO15: track 31.3 -> 39.5 mm, vias 3 -> 1
- net /NRPIBOOT: track 66.1 -> 59.5 mm
- net /USBH_DM: track 16.4 -> 22.4 mm, vias 0 -> 3
- net /GPIO18: track 32.3 -> 26.3 mm
- net /GPIO14: track 28.3 -> 33.8 mm
- net /CC2: track 67.7 -> 72.7 mm
- net /USBH_VBUS: track 54.2 -> 49.4 mm, vias 2 -> 0
- net /GPIO27: track 33.6 -> 38.1 mm, vias 1 -> 3
- net /GPIO17: track 39.3 -> 35.6 mm
- net /ID_SD: track 52.4 -> 56.0 mm
- net /PI_LED_NPWR: track 35.9 -> 32.4 mm
- net /GPIO11: track 49.3 -> 52.6 mm
- net +3V3: track 230.2 -> 232.9 mm, vias 8 -> 6
- net /SD_CMD: track 54.3 -> 51.9 mm
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