File: boards/eos/eos-cm5-base/hardware/eos-cm5-base.kicad_pcb (KiCad board)
At the start: 4 copper layers, 90 x 80 mm, 36 parts, among them J1 CM5 1-100, J2 CM5 101-200, J3 USB-C, J4 USB-A, J5 TRJG0926HENL, J6 microSD, J7 GPIO, J8 FAN, J9 BOOT, SW1 POWER, U1 USBLC6-2SC6, U2 TPS2051C, U3 USBLC6-2SC6, U4 TPD4EUSB30, U5 TPD4EUSB30, U6 RT9742GGJ5

Commit message: fix(boards): rebuild EoS boards without vias in pads
Co-authored-by: Cursor <cursoragent@cursor.com>
Routing:
- net /FAN_PWM: track 94.2 -> 69.6 mm, vias 2 -> 4
- net /EEPROM_NWP: track 75.8 -> 54.8 mm, vias 2 -> 1
- net /GPIO13: track 69.4 -> 51.7 mm, vias 1 -> 2
- net /USBH_VBUS: track 45.1 -> 34.1 mm, vias 2 -> 3
- net GND: track 79.9 -> 88.8 mm, vias 476 -> 422
- net /GPIO10: track 45.4 -> 36.9 mm, vias 1 -> 2
- net /ID_SD: track 55.7 -> 47.3 mm, vias 1 -> 2
- net /CC1: track 56.0 -> 48.1 mm, vias 4 -> 2
- net /CC2: track 62.5 -> 54.9 mm
- net /GPIO8: track 36.4 -> 44.0 mm
- net /NRPIBOOT: track 66.4 -> 58.9 mm
- net /GPIO27: track 33.2 -> 40.3 mm
- net /GPIO9: track 51.7 -> 57.5 mm, vias 1 -> 3
- net /GPIO6: track 60.1 -> 54.4 mm
- net /GPIO5: track 57.8 -> 52.2 mm
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