File: boards/eos/eos-kl25-board/hardware/eos-kl25-board.kicad_pcb (KiCad board)
At the start: 2 copper layers, 68.6 x 53.3 mm, 82 parts, among them J1 USB-C, J2 USB-C, J3 D8-SCL, J4 D0-D7, J5 POWER, J6 A0-A5, J7 SWD, J8 EXT, Q1 AO3400A, Q2 AO3400A, Q3 AO3400A, SW1 RESET, U1 SP0503BAHTG, U2 SP0503BAHTG, U3 TPS2116, U4 AP7361C-33, U5 MKL25Z128VLK4, U6 CP2102N-A02-GQFN20, U7 LIS2HH12, Y1 8MHz

Commit message: fix(boards): rebuild EoS boards without vias in pads
Co-authored-by: Cursor <cursoragent@cursor.com>
Routing:
- net /D1: track 83.6 -> 58.3 mm, vias 2 -> 0
- net +3V3: track 180.9 -> 195.7 mm, vias 9 -> 15
- net /EXT_PTB8: track 19.9 -> 32.4 mm, vias 1 -> 0
- net /EXT_PTE30: track 37.8 -> 26.8 mm
- net /EXT_PTC0: track 20.2 -> 10.1 mm, vias 3 -> 1
- net /RESET: track 49.6 -> 59.6 mm, vias 2 -> 3
- net /A3: track 35.9 -> 44.8 mm
- net /AREF: track 38.5 -> 47.4 mm
- net /EXT_PTB16: track 20.6 -> 11.8 mm, vias 0 -> 1
- net +5V: track 53.0 -> 61.8 mm, vias 1 -> 2
- net GND: track 380.8 -> 372.3 mm, vias 144 -> 154
- net /D0: track 74.9 -> 66.9 mm
- net /A4_SDA: track 69.1 -> 75.7 mm
- net /LED_B: track 21.9 -> 17.4 mm, vias 0 -> 2
- net /ACC_SA0: track 8.05 -> 4.07 mm, vias 2 -> 0
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