File: boards/eos/eos-learn-rp2350/hardware/eos-learn-rp2350.kicad_pcb (KiCad board)
At the start: 4 copper layers, 52.6 x 51.6 mm, 53 parts, among them J1 USB-C, J2 GPIO 0-15, J3 Power, GPIO 16-29, J4 SWD, J5 Qwiic, SW1 BOOTSEL, SW2 RUN, U1 RP2350A, U2 USBLC6-2SC6, U3 AP7361C-33, U4 W25Q128JVS, Y1 12MHz

Commit message: fix(boards): rebuild EoS boards without vias in pads
Co-authored-by: Cursor <cursoragent@cursor.com>
Routing:
- net /USB_D+: track 21.3 -> 32.0 mm
- net VBUS: track 14.7 -> 25.4 mm
- net /CC1: track 13.4 -> 8.92 mm
- net /USB_D-: track 22.2 -> 25.9 mm
- net GND: track 51.3 -> 48.8 mm
- net /CC2: track 11.6 -> 10.4 mm
- net +3V3: track 60.4 -> 61.6 mm
- net +5V: track 33.5 -> 34.0 mm
