File: boards/eos/eos-lpc55s69-board/hardware/eos-lpc55s69-board.kicad_pcb (KiCad board)
At the start: 4 copper layers, 68.6 x 53.3 mm, 99 parts, among them J1 USB-C, J2 USB-C, J3 Cortex Debug, J4 D8-SCL, J5 D0-D7, J6 POWER, J7 A0-A5, Q1 BSS138BK, Q2 BSS138BK, Q3 BSS138BK, SW1 RESET, SW2 ISP, SW3 USER, U1 SP0503BAHTG, U2 SP0503BAHTG, U3 TPS2116, U4 TPS7A91, U5 CP2102N-A02-GQFN24, U6 LPC55S69JBD100, Y1 16MHz, Y2 32.768kHz

Commit message: fix(boards): rebuild EoS boards without vias in pads
Co-authored-by: Cursor <cursoragent@cursor.com>
Routing:
- net /ISP_N: track 42.9 -> 61.0 mm
- net /RESETN: track 98.2 -> 82.0 mm, vias 1 -> 0
- net +5V: track 66.5 -> 58.3 mm
- net /SWDIO: track 24.2 -> 30.2 mm
- net /A3: track 32.3 -> 27.2 mm
- net /SWO: track 25.3 -> 30.2 mm, vias 2 -> 0
- net /VDDA: track 17.2 -> 12.9 mm, vias 2 -> 0
- net /LED_G: track 33.5 -> 37.6 mm
- net /SWCLK: track 23.0 -> 20.2 mm
- net /RGB_RK: track 11.2 -> 8.78 mm
- net /RGB_RD: track 6.55 -> 8.70 mm
- net /USER_BTN: track 38.5 -> 36.4 mm
- net /A4: track 31.1 -> 29.7 mm
- net /LED_B: track 24.4 -> 23.2 mm, vias 2 -> 0
- net /A5: track 31.2 -> 30.3 mm
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