File: boards/eos/eos-ra2e1-board/hardware/eos-ra2e1-board.kicad_pcb (KiCad board)
At the start: 2 copper layers, 68.6 x 53.3 mm, 62 parts, among them J1 USB-C, J2 SWD, J3 D8-SCL, J4 D0-D7, J5 POWER, J6 A0-A5, J7 PMOD A, J8 PMOD B, SW1 RESET, SW2 USER, U1 R7FA2E1A92DFM, U2 SP0503BAHTG, U3 CP2102N-A02-GQFN24, U4 TPS7A91, Y1 32.768kHz

Commit message: fix(boards): rebuild EoS boards without vias in pads
Co-authored-by: Cursor <cursoragent@cursor.com>
Routing:
- net /SPI_MOSI: track 70.4 -> 54.9 mm, vias 0 -> 1
- net GND: track 331.0 -> 319.0 mm, vias 114 -> 120
- net /D4: track 37.2 -> 27.1 mm, vias 1 -> 0
- net /A0: track 41.0 -> 31.0 mm
- net /PMODA_CS3: track 35.0 -> 25.1 mm
- net +5V: track 40.0 -> 32.0 mm, vias 1 -> 2
- net /PMODA_INT: track 25.7 -> 31.5 mm, vias 1 -> 0
- net /SPI_SCK: track 56.7 -> 62.3 mm
- net /PMODA_RST: track 35.2 -> 30.1 mm
- net /RES: track 67.4 -> 64.1 mm
- net /MD: track 24.1 -> 27.3 mm
- net /VBUS: track 31.0 -> 28.3 mm
- net /SPI_MISO: track 46.8 -> 49.1 mm
- net +3V3: track 192.7 -> 190.7 mm
- net /D9: track 28.8 -> 30.7 mm
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