File: boards/eos/eos-stm32-64/hardware/eos-stm32-64.kicad_pcb (KiCad board)
At the start: 2 copper layers, 70 x 82.5 mm, 99 parts, among them CN10 CN10, CN5 D8-D15, CN6 POWER, CN7 CN7, CN8 ANALOG, CN9 D0-D7, J1 USB-C, J2 USB-C, J3 Cortex Debug, J4 IDD, U1 STM32F411RET6, U2 CP2102N-A02-GQFN20, U3 AP7361C-33, U4 AP63205, U5 SP0503BAHTG, U6 SP0503BAHTG, Y1 8MHz, Y2 32.768kHz

Commit message: fix(boards): rebuild EoS boards without vias in pads
Co-authored-by: Cursor <cursoragent@cursor.com>
Routing:
- net /VBUS_VCP: track 30.3 -> 31.9 mm, vias 5 -> 6
- net GND: vias 102 -> 101
